Commit message: [Beetle-Art][URDF] make the visual model up for better visualization

File: robots/beetle/urdf/beetle-art.urdf.xacro (robot description, xacro)
@@ -30,5 +30,5 @@
       </inertial>
       <visual>
-        <origin xyz="0 0 0" rpy="1.570796 0 3.141592"/>
+        <origin xyz="0 0 0.063" rpy="1.570796 0 3.141592"/>
         <geometry>
           <mesh filename="package://beetle/urdf/mesh/base_link_beetle_art.dae"/>

Commit message: [Beetle][Control][NMPC]: test the omnidirectional flight in simulation

File: robots/beetle/urdf/beetle-art.urdf.xacro (robot description, xacro)
@@ -155,5 +155,5 @@
     #### gimbal joints ####
     <joint name="gimbal${self}" type="revolute">
-      <limit effort="6.6" lower="-1.57" upper="1.57" velocity="3.0"/>
+      <limit effort="6.6" lower="-2.36" upper="2.36" velocity="3.0"/>
       <parent link="rotor_arm${self}"/>
       <child link="gimbal_link${self}"/>
