Commit message: [ball]: fix the model error of thrust position

File: robots/beetle_omni/urdf/dragon_ball.urdf.xacro (robot description, xacro)
@@ -164,5 +164,5 @@
       <parent link="gimbal_link${self}"/>
       <child link="rotor_parent${self}"/>
-      <origin rpy="0 0 0" xyz="0.0 0.0 0.0"/>
+      <origin rpy="0 0 0" xyz="0.018 0.0 0.0"/>
     </joint>
     #### rotor joint (virtual) ####

File: robots/beetle_omni/urdf/dragon_ball_bi.urdf.xacro (robot description, xacro)
@@ -162,5 +162,5 @@
       <parent link="gimbal_link${self}"/>
       <child link="rotor_parent${self}"/>
-      <origin rpy="0 0 0" xyz="0.0 0.0 0.0"/>
+      <origin rpy="0 0 0" xyz="0.018 0.0 0.0"/>
     </joint>
     #### rotor joint (virtual) ####
