Commit message: [diff] Functional state for differential MPC (especially second-order)
* Optimized integration of cmd input (which is vel) to get actual thrust and angle to command -> standard blind integration also works but this way it has some form feedback and performs better (especially second-order works better since the servo and rotor model are still kept in the model/feedback and not just implicitly through the integration model)

* Added accurate control loop dt computation for cmd integration

* Increased servo time constant to match simulation setup (gimbal has P-gain of 5.0 and damping factor of 0.8 -> t_servo = 0.8/5.0 = 0.16s) instead of old constant 0.048s THIS MADE IT VERY STABLE AND ACCURATE

* Corrected wrench dynamic computation: Instead of using the symbolic state in the jacobian, use the analytical wrench instead, else the Jacobian is simply zero  -> this works well!

* Bugfix order of init calls and base_thrust initialization

* Added input constraints in Python as they are included in C++ as well

* Added num_rotors and num_servos to controllers to allow for arbitrary configurations

* Corrected indexing in Python ref

* Corrected yaml call for second-order

* Added correctly named AD_C config parameter

* Made visualization cleaner and included reference as well as wrench state

File: robots/beetle_omni/urdf/beetle_art_omni.urdf.xacro (robot description, xacro)
@@ -125,5 +125,7 @@
     #### gimbal joints ####
     <joint name="gimbal${self}" type="revolute">
-      <limit effort="6.6" lower="-3.926991" upper="3.926991" velocity="3.0"/>
+      <!-- 12.07.2026 Previously, velocity="3.0" but according to the XC330-T181-T's datasheet
+      it has a no load speed of 104rev/min at 11.1V translating to 5.44rad/s (UNDER NO LOAD!) -->
+      <limit effort="6.6" lower="-3.926991" upper="3.926991" velocity="5.0"/>
       <parent link="rotor_arm${self}"/>
       <child link="gimbal_link${self}"/>
